Commit message: go2 mapping

File: src/go2/go2_description/urdf/go2_description.urdf (robot description, URDF)
Before this commit: robot go2_description, 43 links, 42 joints
Links:
- added link livox_frame, mass 0
Joints:
- added joint livox_frame_joint: type fixed, parent base_link, child livox_frame, origin xyz=0 0 0.15 rpy=0.12 0 0, axis 0 0 0
- joint base_joint: origin xyz=0.0 0.0 0.0 rpy=0 0 0 -> xyz=0.0 0.0 0.16 rpy=0 0 0
- joint utlidar_joint: origin xyz=0.3 0 -0.03 rpy=0.22 -3.00 2.05 -> xyz=0.28 0 -0.0 rpy=0.25 -3.00 2.05

Commit message: Update Go2 mapping and navigation configuration

File: src/go2/go2_description/urdf/go2_description.urdf (robot description, URDF)
Before this commit: robot go2_description, 44 links, 43 joints
Joints:
- joint utlidar_joint: origin xyz=0.28 0 -0.0 rpy=0.25 -3.00 2.05 -> xyz=0.3 0 -0.03 rpy=0.22 -3.00 2.05

Commit message: fix: utlidar, mid360 정렬 수행

File: src/go2/go2_description/urdf/go2_description.urdf (robot description, URDF)
Before this commit: robot go2_description, 44 links, 43 joints
Joints:
- joint base_joint: origin xyz=0.0 0.0 0.16 rpy=0 0 0 -> xyz=0.0 0.0 0.35 rpy=0 0 0
- joint livox_frame_joint: origin xyz=0 0 0.15 rpy=0.12 0 0 -> xyz=0.2 0.1 0.15 rpy=0.12 0 0
- joint utlidar_joint: origin xyz=0.3 0 -0.03 rpy=0.22 -3.00 2.05 -> xyz=0.28945 0 0.00 rpy=0.22 -3.00 2.15

Commit message: fix: tf 정렬 마무리

File: src/go2/go2_description/urdf/go2_description.urdf (robot description, URDF)
Before this commit: robot go2_description, 44 links, 43 joints
Joints:
- joint livox_frame_joint: origin xyz=0.2 0.1 0.15 rpy=0.12 0 0 -> xyz=0.2 0.1 0.05 rpy=0.12 0 0
